Commit message: Packages renamed. Added global bringup.launch.py launch file.

File: stepit_robot/urdf/stepit.urdf.xacro (robot description, xacro)
@@ -1,6 +1,6 @@
 <?xml version="1.0"?>
 <robot name="stepit" xmlns:xacro="http://ros.org/wiki/xacro">
-  <xacro:include filename="$(find stepit_description)/urdf/stepit.xacro" />
-  <xacro:include filename="$(find stepit_description)/urdf/stepit.ros2_control.xacro" />
+  <xacro:include filename="$(find stepit_robot)/urdf/stepit.xacro" />
+  <xacro:include filename="$(find stepit_robot)/urdf/stepit.ros2_control.xacro" />
   <xacro:stepit />
   <xacro:stepit_ros2_control name="stepit_ros2_control" />

File: stepit_robot/urdf/stepit.xacro (robot description, xacro)
@@ -19,5 +19,5 @@
         <origin xyz="0.0 0.0 0.0" rpy="0 0 0" />
         <geometry>
-          <mesh filename="file://$(find stepit_description)/meshes/cylinder.dae" scale="1 1 1" />
+          <mesh filename="file://$(find stepit_robot)/meshes/cylinder.dae" scale="1 1 1" />
         </geometry>
       </visual>
@@ -27,5 +27,5 @@
         <origin xyz="0.0 0.0 0.0" rpy="0 0 0" />
         <geometry>
-          <mesh filename="file://$(find stepit_description)/meshes/cylinder.dae" scale="1 1 1" />
+          <mesh filename="file://$(find stepit_robot)/meshes/cylinder.dae" scale="1 1 1" />
         </geometry>
       </visual>
