Commit message: URDF

File: stepit_description/urdf/stepit.xacro (robot description, xacro)
@@ -2,9 +2,38 @@
 <robot xmlns:xacro="http://ros.org/wiki/xacro">
   <xacro:macro name="stepit">
+    <link name="base_link">
+      <visual>
+        <geometry>
+          <box size="1 1 1" />
+        </geometry>
+      </visual>
+    </link>
+    <link name="link1">
+      <visual>
+        <origin xyz="0 0 0.5" rpy="0 0 0" />
+        <geometry>
+          <cylinder length="1" radius="0.4" />
+        </geometry>
+      </visual>
+    </link>
+    <link name="link2">
+      <visual>
+        <origin xyz="0 0 -0.5" rpy="0 0 0" />
+        <geometry>
+          <cylinder length="1" radius="0.4" />
+        </geometry>
+      </visual>
+    </link>
     <joint name="joint1" type="revolute">
+      <parent link="base_link" />
+      <child link="link1" />
       <axis xyz="0 0 1" />
+      <limit lower="0.0" upper="0.0" effort="0.0" velocity="0.0" />
     </joint>
     <joint name="joint2" type="revolute">
+      <parent link="base_link" />
+      <child link="link2" />
       <axis xyz="0 0 1" />
+      <limit lower="0.0" upper="0.0" effort="0.0" velocity="0.0" />
     </joint>
   </xacro:macro>

Commit message: Added textured mesh to RVIZ as DAE file.

File: stepit_description/urdf/stepit.xacro (robot description, xacro)
@@ -2,27 +2,38 @@
 <robot xmlns:xacro="http://ros.org/wiki/xacro">
   <xacro:macro name="stepit">
+    <material name="base_link_material">
+      <color rgba="0 0 1 1" />
+    </material>
+    <link name="world" />
     <link name="base_link">
-      <visual>
+      <visual name="base_link_visual">
+        <origin xyz="0.0 0 0.05" rpy="0 0 0" />
         <geometry>
-          <box size="1 1 1" />
+          <box size="2 1 0.1" />
         </geometry>
+        <material name="base_link_material" />
       </visual>
     </link>
     <link name="link1">
-      <visual>
-        <origin xyz="0 0 0.5" rpy="0 0 0" />
+      <visual name="link1_visual">
+        <origin xyz="0.5 0 0.15" rpy="0 0 0" />
         <geometry>
-          <cylinder length="1" radius="0.4" />
+          <mesh filename="file://$(find stepit_description)/meshes/cylinder.dae" scale="1 1 1" />
         </geometry>
       </visual>
     </link>
     <link name="link2">
-      <visual>
-        <origin xyz="0 0 -0.5" rpy="0 0 0" />
+      <visual name="link2_visual">
+        <origin xyz="-0.5 0 0.15" rpy="0 0 0" />
         <geometry>
-          <cylinder length="1" radius="0.4" />
+          <mesh filename="file://$(find stepit_description)/meshes/cylinder.dae" scale="1 1 1" />
         </geometry>
       </visual>
     </link>
+    <joint name="base_link_to_world" type="fixed">
+      <parent link="world" />
+      <child link="base_link" />
+      <axis xyz="0 0 1" />
+    </joint>
     <joint name="joint1" type="revolute">
       <parent link="base_link" />

Commit message: Fixed links positions.

File: stepit_description/urdf/stepit.xacro (robot description, xacro)
@@ -17,5 +17,5 @@
     <link name="link1">
       <visual name="link1_visual">
-        <origin xyz="0.5 0 0.15" rpy="0 0 0" />
+        <origin xyz="0.0 0.0 0.0" rpy="0 0 0" />
         <geometry>
           <mesh filename="file://$(find stepit_description)/meshes/cylinder.dae" scale="1 1 1" />
@@ -25,5 +25,5 @@
     <link name="link2">
       <visual name="link2_visual">
-        <origin xyz="-0.5 0 0.15" rpy="0 0 0" />
+        <origin xyz="0.0 0.0 0.0" rpy="0 0 0" />
         <geometry>
           <mesh filename="file://$(find stepit_description)/meshes/cylinder.dae" scale="1 1 1" />
@@ -39,4 +39,5 @@
       <parent link="base_link" />
       <child link="link1" />
+      <origin xyz="0.5 0.0 0.15" rpy="0 0 0" />
       <axis xyz="0 0 1" />
       <limit lower="0.0" upper="0.0" effort="0.0" velocity="0.0" />
@@ -45,4 +46,5 @@
       <parent link="base_link" />
       <child link="link2" />
+      <origin xyz="-0.5 0.0 0.15" rpy="0 0 0" />
       <axis xyz="0 0 1" />
       <limit lower="0.0" upper="0.0" effort="0.0" velocity="0.0" />

Commit message: Added limits to revolute joints and now using Joint State Publisher GUI to control them.

File: stepit_description/urdf/stepit.xacro (robot description, xacro)
@@ -41,5 +41,5 @@
       <origin xyz="0.5 0.0 0.15" rpy="0 0 0" />
       <axis xyz="0 0 1" />
-      <limit lower="0.0" upper="0.0" effort="0.0" velocity="0.0" />
+      <limit lower="-3.14159265358979" upper="3.14159265358979" effort="0.0" velocity="0.0" />
     </joint>
     <joint name="joint2" type="revolute">
@@ -48,5 +48,5 @@
       <origin xyz="-0.5 0.0 0.15" rpy="0 0 0" />
       <axis xyz="0 0 1" />
-      <limit lower="0.0" upper="0.0" effort="0.0" velocity="0.0" />
+      <limit lower="-3.14159265358979" upper="3.14159265358979" effort="0.0" velocity="0.0" />
     </joint>
   </xacro:macro>

Commit message: Robot now appearing in Ignition.

File: stepit_description/urdf/stepit.xacro (robot description, xacro)
@@ -7,4 +7,9 @@
     <link name="world" />
     <link name="base_link">
+      <inertial>
+        <origin xyz="0 0 0" rpy="0 0 0" />
+        <mass value="0.1" />
+        <inertia ixx="0.0001" ixy="0.0" ixz="0.0" iyy="0.0001" iyz="0.0" izz="0.0001" />
+      </inertial>
       <visual name="base_link_visual">
         <origin xyz="0.0 0 0.05" rpy="0 0 0" />
@@ -16,4 +21,9 @@
     </link>
     <link name="link1">
+      <inertial>
+        <origin xyz="0 0 0" rpy="0 0 0" />
+        <mass value="0.1" />
+        <inertia ixx="0.0001" ixy="0.0" ixz="0.0" iyy="0.0001" iyz="0.0" izz="0.0001" />
+      </inertial>
       <visual name="link1_visual">
         <origin xyz="0.0 0.0 0.0" rpy="0 0 0" />
@@ -24,4 +34,9 @@
     </link>
     <link name="link2">
+      <inertial>
+        <origin xyz="0 0 0" rpy="0 0 0" />
+        <mass value="0.1" />
+        <inertia ixx="0.0001" ixy="0.0" ixz="0.0" iyy="0.0001" iyz="0.0" izz="0.0001" />
+      </inertial>
       <visual name="link2_visual">
         <origin xyz="0.0 0.0 0.0" rpy="0 0 0" />
