Commit message: Updated the code to control 5 stepper motors.

File: stepit_description/urdf/stepit.ros2_control.xacro (robot description, xacro)
@@ -5,5 +5,5 @@
       <hardware>
         <plugin>stepit_hardware/StepitHardware</plugin>
-        <param name="use_dummy">true</param>
+        <param name="use_dummy">false</param>
         <param name="usb_port">/dev/ttyACM0</param>
         <param name="baud_rate">9600</param>
@@ -13,5 +13,5 @@
         <param name="id">0</param>
         <param name="acceleration">3.14159</param>
-        <param name="max_velocity">6.28319</param>
+        <param name="max_velocity">31.4159265358979</param> <!-- 5 rotations/s -->
         <command_interface name="position" />
         <command_interface name="velocity" />
@@ -22,5 +22,32 @@
         <param name="id">1</param>
         <param name="acceleration">3.14159</param>
-        <param name="max_velocity">6.28319</param>
+        <param name="max_velocity">31.4159265358979</param> <!-- 5 rotations/s -->
+        <command_interface name="position" />
+        <command_interface name="velocity" />
+        <state_interface name="position" />
+        <state_interface name="velocity" />
+      </joint>
+      <joint name="joint3">
+        <param name="id">2</param>
+        <param name="acceleration">3.14159</param>
+        <param name="max_velocity">31.4159265358979</param> <!-- 5 rotations/s -->
+        <command_interface name="position" />
+        <command_interface name="velocity" />
+        <state_interface name="position" />
+        <state_interface name="velocity" />
+      </joint>
+      <joint name="joint4">
+        <param name="id">3</param>
+        <param name="acceleration">3.14159</param>
+        <param name="max_velocity">31.4159265358979</param> <!-- 5 rotations/s -->
+        <command_interface name="position" />
+        <command_interface name="velocity" />
+        <state_interface name="position" />
+        <state_interface name="velocity" />
+      </joint>
+      <joint name="joint5">
+        <param name="id">4</param>
+        <param name="acceleration">3.14159</param>
+        <param name="max_velocity">31.4159265358979</param> <!-- 5 rotations/s -->
         <command_interface name="position" />
         <command_interface name="velocity" />

File: stepit_description/urdf/stepit.xacro (robot description, xacro)
@@ -15,5 +15,5 @@
         <origin xyz="0.0 0 0.05" rpy="0 0 0" />
         <geometry>
-          <box size="2 1 0.1" />
+          <box size="5 1 0.1" />
         </geometry>
         <material name="base_link_material" />
@@ -29,5 +29,5 @@
         <origin xyz="0.0 0.0 0.0" rpy="0 0 0" />
         <geometry>
-          <mesh filename="file://$(find stepit_description)/meshes/cylinder.dae" scale="1 1 1" />
+          <mesh filename="file://$(find stepit_description)/meshes/stepper_1.dae" scale="1 1 1" />
         </geometry>
       </visual>
@@ -42,5 +42,44 @@
         <origin xyz="0.0 0.0 0.0" rpy="0 0 0" />
         <geometry>
-          <mesh filename="file://$(find stepit_description)/meshes/cylinder.dae" scale="1 1 1" />
+          <mesh filename="file://$(find stepit_description)/meshes/stepper_2.dae" scale="1 1 1" />
+        </geometry>
+      </visual>
+    </link>
+    <link name="link3">
+      <inertial>
+        <origin xyz="0 0 0" rpy="0 0 0" />
+        <mass value="0.1" />
+        <inertia ixx="0.0001" ixy="0.0" ixz="0.0" iyy="0.0001" iyz="0.0" izz="0.0001" />
+      </inertial>
+      <visual name="link3_visual">
+        <origin xyz="0.0 0.0 0.0" rpy="0 0 0" />
+        <geometry>
+          <mesh filename="file://$(find stepit_description)/meshes/stepper_3.dae" scale="1 1 1" />
+        </geometry>
+      </visual>
+    </link>
+    <link name="link4">
+      <inertial>
+        <origin xyz="0 0 0" rpy="0 0 0" />
+        <mass value="0.1" />
+        <inertia ixx="0.0001" ixy="0.0" ixz="0.0" iyy="0.0001" iyz="0.0" izz="0.0001" />
+      </inertial>
+      <visual name="link4_visual">
+        <origin xyz="0.0 0.0 0.0" rpy="0 0 0" />
+        <geometry>
+          <mesh filename="file://$(find stepit_description)/meshes/stepper_4.dae" scale="1 1 1" />
+        </geometry>
+      </visual>
+    </link>
+    <link name="link5">
+      <inertial>
+        <origin xyz="0 0 0" rpy="0 0 0" />
+        <mass value="0.1" />
+        <inertia ixx="0.0001" ixy="0.0" ixz="0.0" iyy="0.0001" iyz="0.0" izz="0.0001" />
+      </inertial>
+      <visual name="link5_visual">
+        <origin xyz="0.0 0.0 0.0" rpy="0 0 0" />
+        <geometry>
+          <mesh filename="file://$(find stepit_description)/meshes/stepper_5.dae" scale="1 1 1" />
         </geometry>
       </visual>
@@ -54,5 +93,5 @@
       <parent link="base_link" />
       <child link="link1" />
-      <origin xyz="0.5 0.0 0.15" rpy="0 0 0" />
+      <origin xyz="-2.0 0.0 0.15" rpy="0 0 0" />
       <axis xyz="0 0 1" />
       <limit lower="-3.14159265358979" upper="3.14159265358979" effort="0.0" velocity="0.0" />
@@ -61,5 +100,26 @@
       <parent link="base_link" />
       <child link="link2" />
-      <origin xyz="-0.5 0.0 0.15" rpy="0 0 0" />
+      <origin xyz="-1.0 0.0 0.15" rpy="0 0 0" />
+      <axis xyz="0 0 1" />
+      <limit lower="-3.14159265358979" upper="3.14159265358979" effort="0.0" velocity="0.0" />
+    </joint>
+    <joint name="joint3" type="revolute">
+      <parent link="base_link" />
+      <child link="link3" />
+      <origin xyz="0.0 0.0 0.15" rpy="0 0 0" />
+      <axis xyz="0 0 1" />
+      <limit lower="-3.14159265358979" upper="3.14159265358979" effort="0.0" velocity="0.0" />
+    </joint>
+    <joint name="joint4" type="revolute">
+      <parent link="base_link" />
+      <child link="link4" />
+      <origin xyz="1.0 0.0 0.15" rpy="0 0 0" />
+      <axis xyz="0 0 1" />
+      <limit lower="-3.14159265358979" upper="3.14159265358979" effort="0.0" velocity="0.0" />
+    </joint>
+    <joint name="joint5" type="revolute">
+      <parent link="base_link" />
+      <child link="link5" />
+      <origin xyz="2.0 0.0 0.15" rpy="0 0 0" />
       <axis xyz="0 0 1" />
       <limit lower="-3.14159265358979" upper="3.14159265358979" effort="0.0" velocity="0.0" />
