Commit message: Added README file and description file renamed.

File: stepit_description/urdf/stepit.sample_robot.xacro (robot description, xacro)
@@ -1,5 +1,5 @@
 <?xml version="1.0"?>
 <robot xmlns:xacro="http://ros.org/wiki/xacro">
-  <xacro:macro name="stepit">
+  <xacro:macro name="stepit_sample_robot">
     <material name="base_link_material">
       <color rgba="0 0 1 1" />

File: stepit_description/urdf/stepit.urdf.xacro (robot description, xacro)
@@ -1,7 +1,7 @@
 <?xml version="1.0"?>
 <robot name="stepit" xmlns:xacro="http://ros.org/wiki/xacro">
-  <xacro:include filename="$(find stepit_description)/urdf/stepit.xacro" />
+  <xacro:include filename="$(find stepit_description)/urdf/stepit.sample_robot.xacro" />
   <xacro:include filename="$(find stepit_description)/urdf/stepit.ros2_control.xacro" />
-  <xacro:stepit />
+  <xacro:stepit_sample_robot />
   <xacro:stepit_ros2_control name="stepit_ros2_control" />
 </robot>
