Commit message: Ongoing work.

File: freezer_description/urdf/freezer.ros2_control.xacro (robot description, xacro)
@@ -1,8 +1,8 @@
 <?xml version="1.0"?>
 <robot xmlns:xacro="http://www.ros.org/wiki/xacro">
-  <xacro:macro name="stepit_ros2_control" params="name">
+  <xacro:macro name="freezer_ros2_control" params="name">
     <ros2_control name="${name}" type="system">
       <hardware>
-        <plugin>stepit_hardware/StepitHardware</plugin>
+        <plugin>freezer_controller/FreezerController</plugin>
         <param name="use_dummy">true</param>
         <param name="usb_port">/dev/ttyACM0</param>
@@ -10,49 +10,4 @@
         <param name="timeout">2.0</param>
       </hardware>
-      <joint name="joint1">
-        <param name="id">0</param>
-        <param name="acceleration">3.14159</param>
-        <param name="max_velocity">31.4159265358979</param> <!-- 5 rotations/s -->
-        <command_interface name="position" />
-        <command_interface name="velocity" />
-        <state_interface name="position" />
-        <state_interface name="velocity" />
-      </joint>
-      <joint name="joint2">
-        <param name="id">1</param>
-        <param name="acceleration">3.14159</param>
-        <param name="max_velocity">31.4159265358979</param> <!-- 5 rotations/s -->
-        <command_interface name="position" />
-        <command_interface name="velocity" />
-        <state_interface name="position" />
-        <state_interface name="velocity" />
-      </joint>
-      <joint name="joint3">
-        <param name="id">2</param>
-        <param name="acceleration">3.14159</param>
-        <param name="max_velocity">31.4159265358979</param> <!-- 5 rotations/s -->
-        <command_interface name="position" />
-        <command_interface name="velocity" />
-        <state_interface name="position" />
-        <state_interface name="velocity" />
-      </joint>
-      <joint name="joint4">
-        <param name="id">3</param>
-        <param name="acceleration">3.14159</param>
-        <param name="max_velocity">31.4159265358979</param> <!-- 5 rotations/s -->
-        <command_interface name="position" />
-        <command_interface name="velocity" />
-        <state_interface name="position" />
-        <state_interface name="velocity" />
-      </joint>
-      <joint name="joint5">
-        <param name="id">4</param>
-        <param name="acceleration">3.14159</param>
-        <param name="max_velocity">31.4159265358979</param> <!-- 5 rotations/s -->
-        <command_interface name="position" />
-        <command_interface name="velocity" />
-        <state_interface name="position" />
-        <state_interface name="velocity" />
-      </joint>
     </ros2_control>
   </xacro:macro>

Commit message: Fixing freezer connection errors and incorrect freezer control loaded.

File: freezer_description/urdf/freezer.ros2_control.xacro (robot description, xacro)
@@ -4,9 +4,9 @@
     <ros2_control name="${name}" type="system">
       <hardware>
-        <plugin>freezer_controller/FreezerController</plugin>
+        <plugin>freezer_driver/FreezerHardware</plugin>
         <param name="usb_port">/dev/ttyUSB0</param>
         <param name="baud_rate">9600</param>
-        <param name="timeout">1.0</param>
-        <param name="connection_timeout">1.0</param>
+        <param name="timeout">1</param>
+        <param name="connection_timeout">5</param>
       </hardware>
     </ros2_control>

File: freezer_description/urdf/freezer.sample_robot.xacro (robot description, xacro)
@@ -1,5 +1,5 @@
 <?xml version="1.0"?>
 <robot xmlns:xacro="http://ros.org/wiki/xacro">
-  <xacro:macro name="stepit">
+  <xacro:macro name="freezer_sample_robot">
     <material name="base_link_material">
       <color rgba="0 0 1 1" />

File: freezer_description/urdf/freezer.urdf.xacro (robot description, xacro)
@@ -1,7 +1,7 @@
 <?xml version="1.0"?>
 <robot name="freezer" xmlns:xacro="http://ros.org/wiki/xacro">
-  <xacro:include filename="$(find freezer_description)/urdf/freezer.xacro" />
+  <xacro:include filename="$(find freezer_description)/urdf/freezer.sample_robot.xacro" />
   <xacro:include filename="$(find freezer_description)/urdf/freezer.ros2_control.xacro" />
-  <xacro:freezer />
+  <xacro:freezer_sample_robot />
   <xacro:freezer_ros2_control name="freezer_ros2_control" />
 </robot>
